Commit message: Kendi basılabilir parçalar: CadQuery tasarımı, çakışma taraması, sim ölçüleri
- cad/: MG996R/SG90 ölçülerine göre parametrik parçalar (taban, gövde, üst kol,
  ön kol, bilek, tutucu, evolvent dişli çeneler, burçlar); tek ölçü kaynağı
  geometri.py, 142 eklem konumunda katı çakışma taraması (0 çakışma),
  kontrol.py ile 47 tasarım kontrolü, STEP/STL çıktısı
- Simülasyon sayfası artık basılacak parçaların kendisini gösteriyor
  (sim/servo_mesh.js), tutucu ağzı tasarım tablosundan
- Kinematik ölçüler tasarıma geçti: H0 96, L4 95 mm; parça kütleleri hacimden;
  URDF yeniden üretildi; tutucu varsayılan açık açısı 70°
- onshape/onshape_yukle.py: montaj STEP'ini Onshape'e yükler (.env, git'e girmez)
- README: HTM STL satın alma adımı yerine ölçüm + baskı + montaj kılavuzu

Co-Authored-By: Claude Opus 5.5 <noreply@anthropic.com>

File: ros2/servo_kol_description/urdf/servo_kol.urdf (robot description, URDF)
Before this commit: robot servo_kol, 9 links, 8 joints
Links:
- link govde: geometry collision box size=0.04 0.056 0.036; visual box size=0.04 0.056 0.036
- link on_kol: mass 0.058 -> 0.048
- link parmak_sag: mass 0.0175 -> 0.006; geometry collision box size=0.006 0.012 0.0305; visual box size=0.006 0.012 0.0305
- link parmak_sol: mass 0.0175 -> 0.006; geometry collision box size=0.006 0.012 0.0305; visual box size=0.006 0.012 0.0305
- link tutucu_govde: mass 0.034 -> 0.017
- link ust_kol: mass 0.1 -> 0.105
Joints:
- joint j2_omuz: origin xyz=0 0 0.09 rpy=0 0 0 -> xyz=0 0 0.096 rpy=0 0 0
- joint tutucu: limit lower=0.004 upper=0.02 effort=0.11768 velocity=0.05 -> lower=0.0005 upper=0.035 effort=0.11768 velocity=0.05; origin xyz=0 0 0.036 rpy=0 0 0 -> xyz=0 0 0.0645 rpy=0 0 0
- joint tutucu_ayna: limit lower=-0.02 upper=-0.004 effort=0.11768 velocity=0.05 -> lower=-0.035 upper=-0.0005 effort=0.11768 velocity=0.05; origin xyz=0 0 0.036 rpy=0 0 0 -> xyz=0 0 0.0645 rpy=0 0 0
- joint uc_sabit: origin xyz=0 0 0.08 rpy=0 0 0 -> xyz=0 0 0.095 rpy=0 0 0

Commit message: Tasarımı cilala: desteksiz baskı, tornavida erişimi, dayanım ve devrilme kontrolleri
- cad/baski.py: 0,5 mm voksel ile 6 yönde destek analizi (köprü / çıkıntı /
  havada başlayan bölge) ve ışınla en ince duvar; 11/11 parça desteksiz,
  duvarlar >= 1,2 mm
- Üst kol ve ön kol yan yatık basılacak biçimde: düz taban, 45° pahlı uçlar,
  sivri uçlu hafifletme pencereleri (üst kol 84 -> 66 cm³)
- Horn olukları merkez delikten uzaklaştırıldı (0,4-0,9 mm ince et giderildi),
  göbek havşası eklendi; çatal-yanak boşluğu 2 mm (horn yüksekliği belirsizliği)
- J5 yanağı 6 mm, tutucu dişli göbeği tabana sütunla bağlandı
- model.py: montaj sırasına göre 42 vidada tornavida erişimi kontrolü
- kontrol.py: dişli kökü, horn vidası, levha ve burç dayanımı; devrilme hesabı
  (taban vidalanmazsa kol devrilir, belgelendi); 52/52 GEÇTİ
- Simülasyon parça kütleleri ve ağları güncellendi; docs/parcalar.png, montaj.png

Co-Authored-By: Claude Opus 5.5 <noreply@anthropic.com>

File: ros2/servo_kol_description/urdf/servo_kol.urdf (robot description, URDF)
Before this commit: robot servo_kol, 9 links, 8 joints
Links:
- link on_kol: mass 0.048 -> 0.045
- link parmak_sag: mass 0.006 -> 0.007
- link parmak_sol: mass 0.006 -> 0.007
- link tutucu_govde: mass 0.017 -> 0.018

Commit message: Statik mukavemet hesabı; çatal köprüleri 10 mm; Onshape v2
- cad/mukavemet.py + MUKAVEMET.md: CAD kütleleriyle eklem tepkileri (50 g x 1,5
  dinamik, 200 g aşırı yük, servo durma torku), 19 kesit + 7 bağlantı, PLA katman
  içi / katmanlar arası ayrımı (Prusament veri sayfası), emniyet 3, uç sehimi
- Bulgu: eklem momenti çatal köprüsünden burulmayla geçiyor ve yan yatık baskıda
  kayma katmanlar arasına düşüyor; ön kol köprüsünde durma torkunda emniyet ~1,3
  idi. Köprüler 5 -> 10 mm (en kritik kesit artık izin değerinin %69'u)
- Taşıma: 200 g tam uzanıkta kaldırılamaz (omuz durma torkunun %97'si)
- Onshape v2 belgesi: hacimler CadQuery ile birebir, Check interference yalnız
  tasarım gereği horn/mil temasları
- Simülasyon kütleleri, ağlar, görseller ve belgeler güncellendi

Co-Authored-By: Claude Opus 5.5 <noreply@anthropic.com>

File: ros2/servo_kol_description/urdf/servo_kol.urdf (robot description, URDF)
Before this commit: robot servo_kol, 9 links, 8 joints
Links:
- link on_kol: mass 0.045 -> 0.051
- link ust_kol: mass 0.105 -> 0.121
